File: kicad/Biodom.kicad_pcb (KiCad board)
At the start: 2 copper layers, 160 x 99.1 mm, 33 parts, among them J1 Kamera, J15 Display, J16 DC, J17 PWR, J18 RST, J2 Luft, J21 UART, J26 TDO, J27 TDI, J3 Bodentemperatur, J4 Bodenfeuchte, J5 Wasserstand, J6 Lichtstärke, J7 Reserve, J8 Relais, M1 SD-Karte, P1 Spannungsteiler, U1 ESP32

Commit message: .
Parts:
- J7: value Reserve -> Reserve S6
- renumbered M1 to Z2, Z2 to Z4
Changed lines of the file:
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@@
 		(descr "LED, diameter 3.0mm, 2 pins, generated by kicad-footprint-generator")
 		(tags "LED")
-		(property "Reference" "Z2"
+		(property "Reference" "Z4"
 			(at 1.27 -2.96 90)
 			(layer "F.SilkS")
@@
 			)
 		)
-		(property "Value" "Reserve"
+		(property "Value" "Reserve S6"
 			(at -2.54 2.54 0)
 			(layer "F.Fab")
@@
 		(at 157.48 96.52 -90)
 		(descr "Sockel für MicroSD SPI Module")
-		(property "Reference" "M1"
+		(property "Reference" "Z2"
 			(at -5.08 -1.27 90)
 			(unlocked yes)
