File: kicad/Biodom.kicad_sch (KiCad schematic)
At the start: 45 parts, among them J1 Kamera, J10 Lampe2, J11 Heizer, J12 Lüfter, J13 Pumpe, J14 Dunst, J15 Display, J16 DC, J17 PWR, J18 RST, J2 Luft, J21 UART, J24 TMS, J25 TCK, J26 TDO, J27 TDI, J3 Bodentemperatur, J4 Bodenfeuchte, J5 Wasserstand, J6 Lichtstärke, J7 Reserve, J8 Relais, J9 Lampe1, K1 Relais, M1 SD-Karte, P1 Spannungsteiler, U1 ESP32

Commit message: .
Parts:
- J7: value Reserve -> Reserve S6
- renumbered S2 to S1, S3 to S2, S4 to S3, S5 to S4, S6 to S5, M1 to Z2, S1 to Z3, Z2 to Z4
Changed lines of the file:
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@@
 		(on_board no)
 		(dnp no)
-		(property "Reference" "S2"
+		(property "Reference" "S1"
 			(at 157.226 157.226 0)
 			(effects
@@
 			(project ""
 				(path "/dd570807-a3dd-44e3-850a-e9745bc5cfc3"
-					(reference "S2")
+					(reference "S1")
 					(unit 1)
 				)
@@
 		(on_board yes)
 		(dnp no)
-		(property "Reference" "M1"
+		(property "Reference" "Z2"
 			(at 235.712 92.202 0)
 			(effects
@@
 			(project ""
 				(path "/dd570807-a3dd-44e3-850a-e9745bc5cfc3"
-					(reference "M1")
+					(reference "Z2")
 					(unit 1)
 				)
@@
 		(on_board no)
 		(dnp no)
-		(property "Reference" "S3"
+		(property "Reference" "S2"
 			(at 196.85 157.226 0)
 			(effects
@@
 			(project ""
 				(path "/dd570807-a3dd-44e3-850a-e9745bc5cfc3"
-					(reference "S3")
+					(reference "S2")
 					(unit 1)
 				)
@@
 			)
 		)
-		(property "Value" "Reserve"
+		(property "Value" "Reserve S6"
 			(at 135.89 45.466 90)
 			(effects
@@
 		(on_board no)
 		(dnp no)
-		(property "Reference" "S4"
+		(property "Reference" "S3"
 			(at 227.076 156.972 0)
 			(effects
@@
 			(project ""
 				(path "/dd570807-a3dd-44e3-850a-e9745bc5cfc3"
-					(reference "S4")
+					(reference "S3")
 					(unit 1)
 				)
@@
 		(on_board no)
 		(dnp no)
-		(property "Reference" "S6"
+		(property "Reference" "S5"
 			(at 235.712 56.642 0)
 			(effects
@@
 			(project ""
 				(path "/dd570807-a3dd-44e3-850a-e9745bc5cfc3"
-					(reference "S6")
+					(reference "S5")
 					(unit 1)
 				)
@@
 		(on_board yes)
 		(dnp no)
-		(property "Reference" "Z2"
+		(property "Reference" "Z4"
 			(at 181.102 114.3 0)
 			(effects
@@
 			(project ""
 				(path "/dd570807-a3dd-44e3-850a-e9745bc5cfc3"
-					(reference "Z2")
+					(reference "Z4")
 					(unit 1)
 				)
@@
 		(on_board no)
 		(dnp no)
-		(property "Reference" "S5"
+		(property "Reference" "S4"
 			(at 269.748 156.464 0)
 			(effects
@@
 			(project ""
 				(path "/dd570807-a3dd-44e3-850a-e9745bc5cfc3"
-					(reference "S5")
+					(reference "S4")
 					(unit 1)
 				)
@@
 		(on_board no)
 		(dnp no)
-		(property "Reference" "S1"
+		(property "Reference" "Z3"
 			(at 235.712 117.094 0)
 			(effects
@@
 			(project ""
 				(path "/dd570807-a3dd-44e3-850a-e9745bc5cfc3"
-					(reference "S1")
+					(reference "Z3")
 					(unit 1)
 				)
